File: arc-dvi-vidc-skt-brd.kicad_pcb (KiCad board)
At the start: 4 copper layers, 73.6 x 63 mm, 29 parts, among them IC1 SN74ALVC164245, IC2 SN74ALVC164245, IC3 SN74ALVC164245, J1 Connector_50pin_FFC, U1 MIC5219 3.3V

Commit message: Add README, image, licence
Other:
- board text added: "Copyright 2023 Matt Evans CC BY-NC-SA 3.0"
Changed lines of the file:
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@@
     (effects (font (size 1 1) (thickness 0.15)))
+  )
+  (gr_text "Copyright 2023 Matt Evans\n\nCC BY-NC-SA 3.0\n" (at 179.39 171.02) (layer "Cmts.User")
+    (effects (font (size 1 1) (thickness 0.15)) (justify left))
   )
   (segment (start 95.59 123.9075) (end 95.59 123.87) (width 0.4) (layer "F.Cu") (net 1))
