File: arc-dvi-vidc-skt-brd.kicad_sch (KiCad schematic)
At the start: 26 parts, among them IC1 SN74ALVC164245, IC2 SN74ALVC164245, IC3 SN74ALVC164245, J1 Connector_50pin_FFC, U1 MIC5219 3.3V

Commit message: Placed, partially routed
Same schematic as A3000 arc-dvi-vidc-brds, same FFC pinout (yay).
Parts:
- added R1, R2: 4K7, Resistor_SMD:R_0603_1608Metric, symbol Device:R_Small
Connections:
- net +3V3: now also C8.1, R1.1; no longer C7.1
- net +5V: now also C7.1; no longer C8.1
- net CKIN: now also IC3.14 (2B2); no longer IC3.20 (2B6)
- net FLYBK: now also IC3.16 (2B3); no longer IC3.17 (2B4)
- net GND: now also R2.2
- net NHS: now also IC3.22 (2B7); no longer IC3.14 (2B2)
- net NSNDRQ: now also IC3.17 (2B4); no longer IC3.16 (2B3)
- net NVCS: now also IC3.20 (2B6); no longer IC3.13 (2B1)
- net NVIDW: now also IC3.23 (2B8); no longer IC3.12 (1B8)
- net SNDAK: now also IC3.12 (1B8); no longer IC3.22 (2B7)
- net VIDAK: now also IC3.13 (2B1); no longer IC3.23 (2B8)
- net at IC3.30 (2A5): now also RN11.1; no longer RN9.1
- net at J1.41: now also RN11.8 (2); no longer RN9.8 (2)
- net at RN9.3 (1): no longer IC3.27 (2A7)
- net at J1.38: now also RN11.6 (2); no longer RN9.6 (2)
- net at J1.37: now also RN11.5 (2); no longer RN9.5 (2)
- net at J1.39: now also RN11.7 (2); no longer RN9.7 (2)
- net at J1.46: now also RN9.5 (2); no longer RN11.5 (2)
- net ID_DET: now reaches J1.49
- net ID_DET: now also R1.2, R2.1
- net at RN11.3 (1): now also IC3.27 (2A7)
- net at IC3.26 (2A8): now also RN11.4 (1); no longer RN9.4 (1)
- net at RN9.2 (1): no longer IC3.29 (2A6)
- net at IC3.37 (1A8): now also RN9.4 (1); no longer RN11.4 (1)
- net at RN11.2 (1): now also IC3.29 (2A6)
Other:
- note added: "(c) 2023 Matt Evans"
- note added: "A-series version"
- note removed: "(For A3000/soldered VIDC)"
- note removed: "(c) 2021 Matt Evans"
- note removed: "22 Oct 2021"
- moved on the sheet: VIDC_BOT_PLG1, VIDC_TOP_SKT1

Commit message: Add README, image, licence
Other:
- note added: "Copyright 2023 Matt Evans CC BY-NC-SA 3.0"
- note removed: "(c) 2023 Matt Evans"
Changed lines of the file:
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@@
     (effects (font (size 1.778 1.5113)) (justify left bottom))
   )
-  (text "(c) 2023 Matt Evans" (at 535.94 424.18 180)
+  (text "Copyright 2023 Matt Evans\n\nCC BY-NC-SA 3.0" (at 535.94 424.18 180)
     (effects (font (size 1.778 1.5113)) (justify left bottom))
   )
